Commit message: FIX: in transmission tag, replace plugin w/ type for ros2 humble

File: src/smallrobot_description/urdf/smallrobot_macro.xacro (robot description, xacro)
@@ -1,16 +1,18 @@
 <?xml version="1.0"?>
 <robot xmlns:xacro="http://www.ros.org/wiki/xacro" name="smallrobot">
-  <xacro:property name='PI' value='3.14159'/>
+  <xacro:property name='PI' value='3.14159' />
   <xacro:macro name="default_inertial" params="mass">
     <inertial>
-      <mass value="${mass}"/>
+      <mass value="${mass}" />
       <inertia ixx="1.0" ixy="0" ixz="0" iyy="1.0" iyz="0" izz="1.0"/>
+      <!-- for cylinder robort formular in wiki <inertia ixx="${m*(3*r*r+h*h)/12}" ixy="0" ixz="0" iyy="${m*(3*r*r+h*h)/12}" iyz="0"
+        izz="${m*r*r/2}" /> -->
     </inertial>
   </xacro:macro>
   <xacro:macro name="default_transmission" params="number reduction_ratio">
     <transmission name="transmission_${number}">
-      <plugin>transmission_interface/SimpleTransmission</plugin>
+      <type>transmission_interface/SimpleTransmission</type>
       <actuator name="motor_${number}">
-         <mechanicalReduction>${reduction_ratio}</mechanicalReduction>
+        <mechanicalReduction>${reduction_ratio}</mechanicalReduction>
       </actuator>
       <joint name="joint_${number}">
@@ -23,21 +25,21 @@
   <xacro:macro name="default_material">
     <material name="orange">
-      <color rgba="1.0 0.5 0.0 0.8"/>
+      <color rgba="1.0 0.5 0.0 0.8" />
     </material>
   </xacro:macro>
   <xacro:macro name="default_visual" params="xyz rpy size filename">
     <visual>
-      <origin rpy="${rpy}" xyz="${xyz}"/>
+      <origin rpy="${rpy}" xyz="${xyz}" />
       <geometry>
-        <mesh filename="${filename}"/>
+        <mesh filename="${filename}" />
       </geometry>
-      <xacro:default_material name="gray" rgba="1.0 1.0 1.0 0.8"/>
+      <xacro:default_material name="gray" rgba="1.0 1.0 1.0 0.8" />
     </visual>
   </xacro:macro>
   <xacro:macro name="default_collision" params="xyz rpy size filename">
     <collision>
-      <origin rpy="${rpy}" xyz="${xyz}"/>
+      <origin rpy="${rpy}" xyz="${xyz}" />
       <geometry>
-        <mesh filename="${filename}"/>
+        <mesh filename="${filename}" />
       </geometry>
     </collision>
@@ -45,16 +47,17 @@
   <xacro:macro name="default_link" params="name mass xyz rpy size filename">
     <link name="${name}">
-      <xacro:default_inertial mass="${mass}"/>
-      <xacro:default_visual xyz="${xyz}" rpy="${rpy}" size="${size}" filename="${filename}"/>
-      <xacro:default_collision xyz="${xyz}" rpy="${rpy}" size="${size}" filename="${filename}"/>
+      <xacro:default_inertial mass="${mass}" />
+      <xacro:default_visual xyz="${xyz}" rpy="${rpy}" size="${size}" filename="${filename}" />
+      <xacro:default_collision xyz="${xyz}" rpy="${rpy}" size="${size}" filename="${filename}" />
     </link>
   </xacro:macro>
-  <xacro:macro name="default_joint" params="name type parent child xyz rpy axis limit effort lower upper velocity">
+  <xacro:macro name="default_joint"
+    params="name type parent child xyz rpy axis limit effort lower upper velocity">
     <joint name="${name}" type="${type}">
-      <origin rpy="${rpy}" xyz="${xyz}"/>
-      <axis xyz="${axis}"/>
-      <limit effort="${effort}" lower="${lower}" upper="${upper}" velocity="${velocity}"/>
-      <parent link="${parent}"/>
-      <child link="${child}"/>
+      <origin rpy="${rpy}" xyz="${xyz}" />
+      <axis xyz="${axis}" />
+      <limit effort="${effort}" lower="${lower}" upper="${upper}" velocity="${velocity}" />
+      <parent link="${parent}" />
+      <child link="${child}" />
     </joint>
   </xacro:macro>

Commit message: FIX: joint$_ with joint$ in transmssion tag

File: src/smallrobot_description/urdf/smallrobot_macro.xacro (robot description, xacro)
@@ -14,5 +14,5 @@
          <mechanicalReduction>${reduction_ratio}</mechanicalReduction>
       </actuator>
-      <joint name="joint_${number}">
+      <joint name="joint${number}">
         <hardwareInterface>hardware_interface/position</hardwareInterface>
         <!-- <hardwareInterface>hardware_interface/velocity</hardwareInterface>
