Commit message: ADD: gazebo reference='base_link

File: src/smallrobot_description/urdf/smallrobot_gazebo.xacro (robot description, xacro)
@@ -8,4 +8,7 @@
             <parameters>$(find robotarm_controller)/config/robotarm_controllers.yaml</parameters>
         </plugin>
+    </gazebo>
+    <gazebo reference='base_link'>
+        <material>Gazebo/White</material>
     </gazebo>
     <gazebo reference="link1">

Commit message: ADD: base_link and remove parameters tag, coz yaml load frm launch, on gazebo.xacro. s1.ino

File: src/smallrobot_description/urdf/smallrobot_gazebo.xacro (robot description, xacro)
@@ -6,8 +6,8 @@
             <robot_param_node>robot_state_publisher</robot_param_node>
             <!-- <parameters>/home/roach/ros2_ws/install/robotarm_controller/share/robotarm_controller/config/robotarm_controllers.yaml</parameters> -->
-            <parameters>$(find robotarm_controller)/config/robotarm_controllers.yaml</parameters>
+            <!-- <parameters>$(find robotarm_controller)/config/robotarm_controllers.yaml</parameters> -->
         </plugin>
     </gazebo>
-    <gazebo reference='base_link'>
+    <gazebo reference="base_link">
         <material>Gazebo/White</material>
     </gazebo>

File: src/smallrobot_description/urdf/smallrobot_macro.xacro (robot description, xacro)
@@ -5,6 +5,7 @@
     <inertial>
       <mass value="${mass}" />
-      <inertia ixx="1.0" ixy="0" ixz="0" iyy="1.0" iyz="0" izz="1.0"/>
-      <!-- for cylinder robort formular in wiki <inertia ixx="${m*(3*r*r+h*h)/12}" ixy="0" ixz="0" iyy="${m*(3*r*r+h*h)/12}" iyz="0"
+      <inertia ixx="1.0" ixy="0" ixz="0" iyy="1.0" iyz="0" izz="1.0" />
+      <!-- for cylinder robort formular in wiki <inertia ixx="${m*(3*r*r+h*h)/12}" ixy="0" ixz="0"
+      iyy="${m*(3*r*r+h*h)/12}" iyz="0"
         izz="${m*r*r/2}" /> -->
     </inertial>

Commit message: FIX: replace joint name="joint$_{number}" with joint${number} to match settings in yaml

File: src/smallrobot_description/urdf/smallrobot_gazebo.xacro (robot description, xacro)
@@ -6,5 +6,5 @@
             <robot_param_node>robot_state_publisher</robot_param_node>
             <!-- <parameters>/home/roach/ros2_ws/install/robotarm_controller/share/robotarm_controller/config/robotarm_controllers.yaml</parameters> -->
-            <!-- <parameters>$(find robotarm_controller)/config/robotarm_controllers.yaml</parameters> -->
+            <parameters>$(find robotarm_controller)/config/robotarm_controllers.yaml</parameters>
         </plugin>
     </gazebo>

File: src/smallrobot_description/urdf/smallrobot_macro.xacro (robot description, xacro)
@@ -17,5 +17,5 @@
         <mechanicalReduction>${reduction_ratio}</mechanicalReduction>
       </actuator>
-      <joint name="joint_${number}">
+      <joint name="joint${number}">
         <hardwareInterface>hardware_interface/position</hardwareInterface>
         <!-- <hardwareInterface>hardware_interface/velocity</hardwareInterface>
