Commit message: ADD: gripper in urdf, yaml and controller.launch. 3 controllers are activated and h/w components are availebl/claimed. however, moveit does not work

File: src/smallrobot_description/urdf/smallrobot.urdf (robot description, URDF)
Before this commit: robot smallrobot, 8 links, 7 joints
Links:
- added link gripper_left; visual mesh filename=package://smallrobot_description/meshes/gripper_left_palm.s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
- added link gripper_right; visual mesh filename=package://smallrobot_description/meshes/gripper_right_palm.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
Joints:
- added joint joint7: type revolute, parent link6, child gripper_right, origin xyz=-0.04 0.13 -0.1 rpy=0 0 0, axis 0 0 1, limit lower=-1.570795 upper=0.0 effort=100 velocity=1.57
- added joint joint8: type revolute, parent link6, child gripper_left, origin xyz=-0.22 0.13 -0.1 rpy=0 0 0, axis 0 0 1 , limit lower=0.0 upper=1.570795 effort=100 velocity=1.57, mimic joint=joint7 multiplier=-1

File: src/smallrobot_description/urdf/smallrobot.urdf.xacro (robot description, xacro)
@@ -7,6 +7,7 @@
 <robot xmlns:xacro="http://www.ros.org/wiki/xacro" name="smallrobot">
   <!-- PI & is_sim will be accessible from included xacro files -->
-  <xacro:arg name='is_sim'
-    default='true' />
+  <xacro:arg name='is_sim' default='true' />
+  <xacro:arg name="use_fake_hardware" default="false" />
+  <xacro:arg name="fake_sensor_commands" default="false" />
   <xacro:property name='PI' value='3.14159' />
   <xacro:property
@@ -33,5 +34,5 @@
     <xacro:default_inertial mass="1.0" />
     <visual>
-      <origin rpy="0 0 3.1415926" xyz="0.047 0.0121 0.25" />
+      <origin rpy="0 0 ${PI}" xyz="0.047 0.0121 0.25" />
       <geometry>
         <mesh filename="package://smallrobot_description/meshes/link1.STL" />
@@ -41,5 +42,5 @@
     </visual>
     <collision>
-      <origin rpy="0 0 3.1415926" xyz="0.047 0.0121 0.25" />
+      <origin rpy="0 0 ${PI}" xyz="0.047 0.0121 0.25" />
       <geometry>
         <mesh filename="package://smallrobot_description/meshes/link1.STL" />
@@ -51,5 +52,5 @@
     <origin rpy="0 0 0" xyz="0 0 0.043" />
     <axis xyz="0 0 1" />
-    <limit effort="100" lower="-2.0" upper="2.0" velocity="1.57" />
+    <limit effort="100" lower="-2.0" upper="2.0" velocity="4.8" />
     <parent link="base_link" />
     <child link="link1" />
@@ -58,5 +59,5 @@
     <xacro:default_inertial mass="0.5" />
     <visual>
-      <origin rpy="0 0 3.1415926" xyz="0.047 0.012 0.208" />
+      <origin rpy="0 0 ${PI}" xyz="0.047 0.012 0.208" />
       <geometry>
         <mesh filename="package://smallrobot_description/meshes/link2.STL" />
@@ -65,5 +66,5 @@
     </visual>
     <collision>
-      <origin rpy="0 0 3.1415926" xyz="0.047 0.012 0.208" />
+      <origin rpy="0 0 ${PI}" xyz="0.047 0.012 0.208" />
       <geometry>
         <mesh filename="package://smallrobot_description/meshes/link2.STL" />
@@ -75,5 +76,5 @@
     <origin rpy="0 0 0" xyz="0.047 -0.0485 0.098" />
     <axis xyz="0 1 0" />
-    <limit effort="100" lower="-1.5707963" upper="3.1415926" velocity="1.57" />
+    <limit effort="100" lower="-${PI/2}" upper="${PI}" velocity="4.8" />
     <parent link="link1" />
     <child link="link2" />
@@ -82,5 +83,5 @@
     <xacro:default_inertial mass="0.3" />
     <visual>
-      <origin rpy="1.5707963 0 3.1415926" xyz="0 0 0" />
+      <origin rpy="${PI/2} 0 ${PI}" xyz="0 0 0" />
       <geometry>
         <mesh filename="package://smallrobot_description/meshes/link3.STL" />
@@ -89,5 +90,5 @@
     </visual>
     <collision>
-      <origin rpy="1.5707963 0 3.1415926" xyz="0 0 0" />
+      <origin rpy="${PI/2} 0 ${PI}" xyz="0 0 0" />
       <geometry>
         <mesh filename="package://smallrobot_description/meshes/link3.STL" />
@@ -99,5 +100,5 @@
     <origin rpy="0 0 0" xyz="0 0.08 0.111" />
     <axis xyz="0 1 0" />
-    <limit effort="100" lower="-3.1415926" upper="1.5707963" velocity="1.57" />
+    <limit effort="100" lower="-${PI}" upper="${PI/2}" velocity="4.8" />
     <parent link="link2" />
     <child link="link3" />
@@ -106,5 +107,5 @@
     <xacro:default_inertial mass="0.1" />
     <visual>
-      <origin rpy="0 0 3.1415926" xyz="0.08 -0.0286 0.01" />
+      <origin rpy="0 0 ${PI}" xyz="0.08 -0.0286 0.01" />
       <geometry>
         <mesh filename="package://smallrobot_description/meshes/link4.STL" />
@@ -113,5 +114,5 @@
     </visual>
     <collision>
-      <origin rpy="0 0 3.1415926" xyz="0.08 -0.0286 0.01" />
+      <origin rpy="0 0 ${PI}" xyz="0.08 -0.0286 0.01" />
       <geometry>
         <mesh filename="package://smallrobot_description/meshes/link4.STL" />
@@ -121,7 +122,7 @@
   <joint
     name="joint4" type="revolute">
-    <origin rpy="0 1.5707963 0" xyz="-0.026 -0.0316 0.0258" />
+    <origin rpy="0 ${PI/2} 0" xyz="-0.026 -0.0316 0.0258" />
     <axis xyz="0 0 1" />
-    <limit effort="100" lower="-1.5707963" upper="1.5707963" velocity="1.57" />
+    <limit effort="100" lower="-${PI/2}" upper="${PI/2}" velocity="4.8" />
     <parent link="link3" />
     <child link="link4" />
@@ -130,5 +131,5 @@
     <xacro:default_inertial mass="0.1" />
     <visual>
-      <origin rpy="0 1.5707963 1.5707963" xyz="0.016 0.003 0.106" />
+      <origin rpy="0 ${PI/2} ${PI/2}" xyz="0.016 0.003 0.106" />
       <geometry>
         <mesh filename="package://smallrobot_description/meshes/link5.STL">
@@ -138,5 +139,5 @@
     </visual>
     <collision>
-      <origin rpy="0 1.5707963 1.5707963" xyz="0.016 0.003 0.106" />
+      <origin rpy="0 ${PI/2} ${PI/2}" xyz="0.016 0.003 0.106" />
       <geometry>
         <mesh filename="package://smallrobot_description/meshes/link5.STL" />
@@ -144,9 +145,8 @@
     </collision>
   </link>
-  <joint
-    name="joint5" type="revolute">
-    <origin rpy="0 -1.5707963 0" xyz="0 0 0.144" />
+  <joint name="joint5" type="revolute">
+    <origin rpy="0 -${PI/2} 0" xyz="0 0 0.144" />
     <axis xyz="0 1 0" />
-    <limit effort="100" lower="-3.1415926" upper="3.1415926" velocity="1.57" />
+    <limit effort="100" lower="-${PI}" upper="${PI}" velocity="4.8" />
     <parent link="link4" />
     <child link="link5" />
@@ -155,5 +155,5 @@
     <xacro:default_inertial mass="0.02" />
     <visual>
-      <origin rpy="3.1415926 0 -1.5707963" xyz="0.018 0 0" />
+      <origin rpy="${PI} 0 -${PI/2}" xyz="0.018 0 0" />
       <geometry>
         <mesh filename="package://smallrobot_description/meshes/link6.STL" />
@@ -162,5 +162,5 @@
     </visual>
     <collision>
-      <origin rpy="3.1415926 0 -1.5707963" xyz="0.018 0 0" />
+      <origin rpy="${PI} 0 -${PI/2}" xyz="0.018 0 0" />
       <geometry>
         <mesh filename="package://smallrobot_description/meshes/link6.STL" />
@@ -171,12 +171,12 @@
     <origin rpy="0 0 0" xyz="0.0253 0 0" />
     <axis xyz="1 0 0" />
-    <limit effort="100" lower="-3.1415926" upper="3.1415926" velocity="1.57" />
+    <limit effort="100" lower="-${PI}" upper="${PI}" velocity="4.8" />
     <parent link="link5" />
     <child link="link6" />
   </joint>
   <link name="link6">
-    <!-- <xacro:default_inertial mass="0.01" />
-    <visual>
-      <origin rpy="0 0 3.1415926" xyz="-0.0555 0.003 -0.016" />
+    <xacro:default_inertial mass="0.01" />
+    <visual>
+      <origin rpy="0 0 ${PI}" xyz="-0.0555 0.003 -0.016" />
       <geometry>
         <mesh filename="package://smallrobot_description/meshes/link7.STL" />
@@ -185,13 +185,42 @@
     </visual>
     <collision>
-      <origin rpy="0 0 3.1415926" xyz="-0.0555 0.003 -0.016" />
+      <origin rpy="0 0 ${PI}" xyz="-0.0555 0.003 -0.016" />
       <geometry>
         <mesh filename="package://smallrobot_description/meshes/link7.STL" />
       </geometry>
-    </collision> -->
-  </link>
+    </collision>
+  </link>
+  <link name="flange">
+    <inertial>
+      <origin xyz="0 0 0" />
+      <mass value="0.01" />
+      <inertia ixx="1.0e-06" ixy="0.0" ixz="0.0"
+        iyy="1.0e-06" iyz="0.0"
+        izz="1.0e-06" />
+    </inertial>
+    <visual>
+      <origin xyz="0 0 0" rpy="0 0 -${PI/2}" />
+      <geometry>
+        <mesh filename="${meshes_file_direction}/flange.stl" scale="0.001 0.001 0.001" />
+      </geometry>
+      <material name="grey">
+        <color rgba="0.2 0.2 0.2 1" />
+      </material>
+    </visual>
+    <collision>
+      <origin xyz="0 0 0" rpy="0 0 0" />
+      <geometry>
+        <box size="0.01 0.01 0.01" />
+      </geometry>
+    </collision>
+  </link>
+  <joint name="link6_to_flange" type="fixed">
+    <parent link="link6" />
+    <child link="flange" />
+    <origin xyz="0 0 0" rpy="0 0 0" />
+  </joint>
   <joint
     name="gripper_left_joint" type="prismatic">
-    <parent link="link6" />
+    <parent link="flange" />
     <child link="gripper_left_link" />
     <origin xyz="0.0817 0.021 0.0" rpy="0 0 0" />
@@ -225,5 +254,5 @@
   </link>
   <joint name="gripper_right_joint" type="prismatic">
-    <parent link="link6" />
+    <parent link="flange" />
     <child link="gripper_right_link" />
     <origin xyz="0.0817 -0.021 0" rpy="0 0 0" />
@@ -258,4 +287,5 @@
     </inertial>
   </link>
+  <!--
   <joint name="end_effector_joint" type="fixed">
     <parent link="link6" />
@@ -273,5 +303,5 @@
       </material>
     </visual>
-  </link>
+  </link> -->
   <!-- <link name="ee_link" />
   <joint name="ee_fixed" type="fixed">
@@ -280,9 +310,11 @@
     <origin xyz="0 0 0.1" rpy="0 0 0" />
   </joint> -->
-  <xacro:default_transmission number='1' reduction_ratio='4.8' />
-  <xacro:default_transmission number='2' reduction_ratio='4.0' />
-  <xacro:default_transmission number='3' reduction_ratio='5.0' />
-  <xacro:default_transmission number='4' reduction_ratio='2.8' />
-  <xacro:default_transmission number='5' reduction_ratio='2.1' />
-  <xacro:default_transmission number='6' reduction_ratio='1.0' />
+  <xacro:default_transmission idx='1' joint_name='joint1' reduction_ratio='4.8' />
+  <xacro:default_transmission idx='2' joint_name='joint2' reduction_ratio='4.0' />
+  <xacro:default_transmission idx='3' joint_name='joint3' reduction_ratio='5.0' />
+  <xacro:default_transmission idx='4' joint_name='joint4' reduction_ratio='2.8' />
+  <xacro:default_transmission idx='5' joint_name='joint5' reduction_ratio='2.1' />
+  <xacro:default_transmission idx='6' joint_name='joint6' reduction_ratio='1.0' />
+  <xacro:default_transmission idx='7' joint_name='gripper_left_joint' reduction_ratio='1.0' />
+  <xacro:default_transmission idx='8' joint_name='gripper_right_joint' reduction_ratio='1.0' />
 </robot>

File: src/smallrobot_description/urdf/smallrobot_gazebo.xacro (robot description, xacro)
@@ -30,3 +30,9 @@
         <material>Gazebo/Orange</material>
     </gazebo>
+    <gazebo reference="gripper_left_link">
+        <material>Gazebo/Grey</material>
+    </gazebo>
+     <gazebo reference="gripper_right_link">
+        <material>Gazebo/Grey</material>
+    </gazebo>
 </robot>

File: src/smallrobot_description/urdf/smallrobot_macro.xacro (robot description, xacro)
@@ -11,14 +11,14 @@
     </inertial>
   </xacro:macro>
-  <xacro:macro name="default_transmission" params="number reduction_ratio">
-    <transmission name="transmission_${number}">
+  <xacro:macro name="default_transmission" params="idx joint_name reduction_ratio">
+    <transmission name="transmission_${idx}">
       <type>transmission_interface/SimpleTransmission</type>
-      <actuator name="motor_${number}">
+      <actuator name="motor_${idx}">
         <mechanicalReduction>${reduction_ratio}</mechanicalReduction>
       </actuator>
-      <joint name="joint${number}">
+      <joint name="${joint_name}">
         <hardwareInterface>hardware_interface/position</hardwareInterface>
-        <!-- <hardwareInterface>hardware_interface/velocity</hardwareInterface>
-        <hardwareInterface>hardware_interface/effort</hardwareInterface> -->
+        <hardwareInterface>hardware_interface/velocity</hardwareInterface>
+        <!-- <hardwareInterface>hardware_interface/effort</hardwareInterface> --> -->
       </joint>
     </transmission>

File: src/smallrobot_description/urdf/smallrobot_ros2_control.xacro (robot description, xacro)
@@ -64,4 +64,22 @@
       <state_interface name="velocity"/>
     </joint>
+    <joint name="gripper_left_joint">
+      <command_interface name="position">
+        <param name='min'>-0.01</param>
+        <param name='max'>0.019</param>
+      </command_interface>
+      <state_interface name="position" />
+      <!-- <state_interface name="velocity"/> -->
+    </joint>
+    <joint name="gripper_right_joint">
+      <!-- <param name='mimic'>gripper_left_joint</param>
+      <param name='multiplier'>1.0</param> -->
+      <command_interface name="position">
+        <param name='min'>-0.01</param>
+        <param name='max'>0.019</param>
+      </command_interface>
+      <state_interface name="position" />
+      <!-- <state_interface name="velocity"/> -->
+    </joint>
   </ros2_control>
 </robot>
