Commit message: FIX: remove name for rviz in moveit.launch to avoid multiple instance of rviz.standardize gazebo.launch. give up gazebo as alway fails coz of <base_class_type='hardware_interface::SystemInterface'> issue

File: src/smallrobot_description/urdf/generated_robot.urdf (robot description, URDF)
Before this commit: robot smallrobot, 12 links, 11 joints
Joints:
- joint gripper_left_joint: limit lower=-0.010 upper=0.019 effort=1000 velocity=4.8 -> lower=-0.010 upper=0.019 effort=10 velocity=04.8
- joint gripper_right_joint: limit lower=-0.010 upper=0.019 effort=1000 velocity=4.8 -> lower=-0.010 upper=0.019 effort=10 velocity=04.8
- joint joint1: limit lower=-2.0 upper=2.0 effort=100 velocity=4.8 -> lower=-2.0 upper=2.0 effort=10 velocity=4.8
- joint joint2: limit lower=-1.570795 upper=3.14159 effort=100 velocity=4.8 -> lower=-1.570795 upper=3.14159 effort=10 velocity=4.8
- joint joint3: limit lower=-3.14159 upper=1.570795 effort=100 velocity=4.8 -> lower=-3.14159 upper=1.570795 effort=10 velocity=4.8
- joint joint4: limit lower=-1.570795 upper=1.570795 effort=100 velocity=4.8 -> lower=-1.570795 upper=1.570795 effort=10 velocity=4.8
- joint joint5: limit lower=-3.14159 upper=3.14159 effort=100 velocity=4.8 -> lower=-3.14159 upper=3.14159 effort=10 velocity=4.8
- joint joint6: limit lower=-3.14159 upper=3.14159 effort=100 velocity=4.8 -> lower=-3.14159 upper=3.14159 effort=10 velocity=4.8

File: src/smallrobot_description/urdf/smallrobot.urdf.xacro (robot description, xacro)
@@ -52,5 +52,5 @@
     <origin rpy="0 0 0" xyz="0 0 0.043" />
     <axis xyz="0 0 1" />
-    <limit effort="100" lower="-2.0" upper="2.0" velocity="4.8" />
+    <limit acceleration="2.0" effort="10" lower="-2.0" upper="2.0" velocity="4.8" />
     <parent link="base_link" />
     <child link="link1" />
@@ -76,5 +76,5 @@
     <origin rpy="0 0 0" xyz="0.047 -0.0485 0.098" />
     <axis xyz="0 1 0" />
-    <limit effort="100" lower="-${PI/2}" upper="${PI}" velocity="4.8" />
+    <limit acceleration="2.0" effort="10" lower="-${PI/2}" upper="${PI}" velocity="4.8" />
     <parent link="link1" />
     <child link="link2" />
@@ -100,5 +100,5 @@
     <origin rpy="0 0 0" xyz="0 0.08 0.111" />
     <axis xyz="0 1 0" />
-    <limit effort="100" lower="-${PI}" upper="${PI/2}" velocity="4.8" />
+    <limit acceleration="2.0" effort="10" lower="-${PI}" upper="${PI/2}" velocity="4.8"/>
     <parent link="link2" />
     <child link="link3" />
@@ -124,5 +124,5 @@
     <origin rpy="0 ${PI/2} 0" xyz="-0.026 -0.0316 0.0258" />
     <axis xyz="0 0 1" />
-    <limit effort="100" lower="-${PI/2}" upper="${PI/2}" velocity="4.8" />
+    <limit acceleration="2.0" effort="10" lower="-${PI/2}" upper="${PI/2}" velocity="4.8" />
     <parent link="link3" />
     <child link="link4" />
@@ -148,5 +148,5 @@
     <origin rpy="0 -${PI/2} 0" xyz="0 0 0.144" />
     <axis xyz="0 1 0" />
-    <limit effort="100" lower="-${PI}" upper="${PI}" velocity="4.8" />
+    <limit acceleration="2.0" effort="10" lower="-${PI}" upper="${PI}" velocity="4.8" />
     <parent link="link4" />
     <child link="link5" />
@@ -171,5 +171,5 @@
     <origin rpy="0 0 0" xyz="0.0253 0 0" />
     <axis xyz="1 0 0" />
-    <limit effort="100" lower="-${PI}" upper="${PI}" velocity="4.8" />
+    <limit acceleration="2.0" effort="10" lower="-${PI}" upper="${PI}" velocity="4.8" />
     <parent link="link5" />
     <child link="link6" />
@@ -226,5 +226,5 @@
     <origin xyz="0.0817 0.021 0.0" rpy="0 0 0" />
     <axis xyz="0 1 0" />
-    <limit velocity="4.8" effort="1000" lower="-0.010" upper="0.019" />
+    <limit acceleration="2.0" velocity="04.8" effort="10" lower="-0.010" upper="0.019" />
     <dynamics damping="0.1" />
   </joint>
@@ -258,5 +258,5 @@
     <origin xyz="0.0817 -0.021 0" rpy="0 0 0" />
     <axis xyz="0 -1 0" />
-    <limit velocity="4.8" effort="1000" lower="-0.010" upper="0.019" />
+    <limit acceleration="2.0" velocity="04.8" effort="10" lower="-0.010" upper="0.019" />
     <dynamics damping="0.7" />
     <mimic joint="gripper_left_joint" multiplier="1" />

File: src/smallrobot_description/urdf/smallrobot_gazebo.xacro (robot description, xacro)
@@ -1,4 +1,5 @@
 <?xml version="1.0"?>
 <robot xmlns:xacro="http://www.ros.org/wiki/xacro" name="smallrobot" params="number">
+    <xacro:macro name='smallrobot_gazebo'>
     <xacro:macro name="default_transmission" params="idx joint_name reduction_ratio">
         <transmission name="transmission_${idx}">
@@ -14,11 +15,4 @@
         </transmission>
     </xacro:macro>
-    <gazebo>
-        <plugin filename="gz_ros2_control-system" name="gz_ros2_control::GazeboSimROS2ControlPlugin">
-            <!-- <robot_param>robot_description</robot_param>
-            <robot_param_node>robot_state_publisher</robot_param_node>   -->
-            <parameters>$(find robotarm_controller)/config/sim_controllers.yaml</parameters>
-        </plugin>
-    </gazebo>
     <gazebo reference="base_link">
         <material>Gazebo/White</material>
@@ -59,3 +53,15 @@
     <xacro:default_transmission idx='7' joint_name='gripper_left_joint' reduction_ratio='1.0' />
     <xacro:default_transmission idx='8' joint_name='gripper_right_joint' reduction_ratio='1.0' />
+    <!-- <ros2_control name="GazeboSimSystem" type="system">
+        <hardware>
+            <plugin>gz_ros2_control/GazeboSimSystem</plugin>
+        </hardware>
+    </ros2_control> -->
+    <gazebo>
+        <plugin name="gz_ros2_control::GazeboSimROS2ControlPlugin" filename="libgz_ros2_control-system">
+            <parameters>$(find robotarm_controller)/config/sim_controllers.yaml</parameters>
+            <!-- <controller_manager_prefix_node_name>controller_manager</controller_manager_prefix_node_name> -->
+        </plugin>
+    </gazebo>
+    </xacro:macro>
 </robot>

File: src/smallrobot_description/urdf/smallrobot_ros2_control.xacro (robot description, xacro)
@@ -6,6 +6,5 @@
     <xacro:if value="$(arg is_sim)">
        <hardware>
-          <!-- <plugin>gz_ros2_control/GazeboSimSystem</plugin> -->
-          <plugin>mock_components/GenericSystem</plugin>
+          <plugin>gz_ros2_control/GazeboSimSystem</plugin>
         </hardware>
     </xacro:if>
