Commit message: ADD:h/w interface, robotarm_interface.xml. MODIFY:urdf.xacro, control.xacro, controller.luanch.py. So we can choose sim or real robot by passing argis_sim on launching controller.launch.py

File: src/smallrobot_description/urdf/smallrobot.urdf.xacro (robot description, xacro)
@@ -5,6 +5,12 @@
 <!-- =================================================================================== -->
 <robot xmlns:xacro="http://www.ros.org/wiki/xacro" name="smallrobot">
+  <!-- PI & is_sim will be accessible from included xacro files -->
+  <xacro:arg name='is_sim' default='true'/>
+  <xacro:property name='PI' value='3.14159' />
+  <!-- include gazebo parameters -->
   <xacro:include filename="$(find smallrobot_description)/urdf/smallrobot_gazebo.xacro" />
+  <!-- include ros2_control plugins -->
   <xacro:include filename="$(find smallrobot_description)/urdf/smallrobot_ros2_control.xacro"/>
+  <!-- useful macros -->
   <xacro:include filename="$(find smallrobot_description)/urdf/smallrobot_macro.xacro"/>
   <link name="world"/>

File: src/smallrobot_description/urdf/smallrobot_ros2_control.xacro (robot description, xacro)
@@ -1,10 +1,18 @@
 <?xml version="1.0"?>
 <robot xmlns:xacro="http://www.ros.org/wiki/xacro" name="smallrobot">
-  <xacro:property name='PI' value='3.14159'/>
   <ros2_control name="smallrobot_hw" type="system">
-    <hardware>
-      <!-- <plugin>ros2_control_demo_hardware/GenericSystem</plugin> -->
-      <plugin>gazebo_ros2_control/GazeboSystem</plugin>
-    </hardware>
+    <!-- ros2_control gazebo simulator-->
+    <xacro:if value="${is_sim}">
+      <hardware>
+        <plugin>gazebo_ros2_control/GazeboSystem</plugin>
+      </hardware>
+    </xacro:if>
+    <!-- ros2_control real robot hw interface-->
+    <xacro:unless value="${arg is_sim}">
+      <hardware>
+        <plugin>robotarm_controller/RobotArmInterface</plugin>
+        <param name='port'>/dev/ttyUSB0</param>
+      </hardware>
+    </xacro:unless>
     <joint name="joint1">
       <command_interface name="position">
@@ -12,5 +20,5 @@
         <param name='max'>${PI}/2</param>
       </command_interface>
-      <state_interface name="position"/>
+      <state_interface name="position" />
     </joint>
     <joint name="joint2">
@@ -19,5 +27,5 @@
         <param name='max'>${PI}/2</param>
       </command_interface>
-      <state_interface name="position"/>
+      <state_interface name="position" />
     </joint>
     <joint name="joint3">
@@ -26,5 +34,5 @@
         <param name='max'>${PI}/2</param>
       </command_interface>
-      <state_interface name="position"/>
+      <state_interface name="position" />
     </joint>
     <joint name="joint4">
@@ -33,5 +41,5 @@
         <param name='max'>${PI}/2</param>
       </command_interface>
-      <state_interface name="position"/>
+      <state_interface name="position" />
     </joint>
     <joint name="joint5">
@@ -40,5 +48,5 @@
         <param name='max'>${PI}/2</param>
       </command_interface>
-      <state_interface name="position"/>
+      <state_interface name="position" />
     </joint>
     <joint name="joint6">
@@ -47,5 +55,5 @@
         <param name='max'>${PI}/2</param>
       </command_interface>
-      <state_interface name="position"/>
+      <state_interface name="position" />
     </joint>
   </ros2_control>

Commit message: add RL capbility

File: src/smallrobot_description/urdf/smallrobot.urdf.xacro (robot description, xacro)
@@ -1,185 +1,192 @@
 <?xml version="1.0"?>
 <!-- =================================================================================== -->
-<!-- |    This document was autogenerated by xacro from /home/roach/ros2_ws/src/smallrobot_description/urdf/smallrobot_description.xacro | -->
+<!-- |    This document was autogenerated by xacro from
+/home/roach/ros2_ws/src/smallrobot_description/urdf/smallrobot_description.xacro | -->
 <!-- |    EDITING THIS FILE BY HAND IS NOT RECOMMENDED                                 | -->
 <!-- =================================================================================== -->
 <robot xmlns:xacro="http://www.ros.org/wiki/xacro" name="smallrobot">
   <!-- PI & is_sim will be accessible from included xacro files -->
-  <xacro:arg name='is_sim' default='true'/>
+  <xacro:arg name='is_sim' default='true' />
   <xacro:property name='PI' value='3.14159' />
   <!-- include gazebo parameters -->
   <xacro:include filename="$(find smallrobot_description)/urdf/smallrobot_gazebo.xacro" />
   <!-- include ros2_control plugins -->
-  <xacro:include filename="$(find smallrobot_description)/urdf/smallrobot_ros2_control.xacro"/>
+  <xacro:include filename="$(find smallrobot_description)/urdf/smallrobot_ros2_control.xacro" />
   <!-- useful macros -->
-  <xacro:include filename="$(find smallrobot_description)/urdf/smallrobot_macro.xacro"/>
-  <link name="world"/>
+  <xacro:include filename="$(find smallrobot_description)/urdf/smallrobot_macro.xacro" />
+  <link name="world" />
   <!-- Fixed joint from world to base_link -->
   <joint name="world_to_base" type="fixed">
-    <origin xyz="0 0 0" rpy="0 0 0"/>
-    <parent link="world"/>
-    <child link="base_link"/>
+    <origin xyz="0 0 0" rpy="0 0 0" />
+    <parent link="world" />
+    <child link="base_link" />
   </joint>
   <link name="base_link">
-    <xacro:default_inertial mass="1.0"/>
+    <xacro:default_inertial mass="1.0" />
     <visual>
-      <origin rpy="0 0 3.1415926" xyz="0.047 0.0121 0.25"/>
+      <origin rpy="0 0 3.1415926" xyz="0.047 0.0121 0.25" />
       <geometry>
-        <mesh filename="package://smallrobot_description/meshes/link1.STL"/>
+        <mesh filename="package://smallrobot_description/meshes/link1.STL" />
         <!-- <box size="0.5 0.5 0.5"/> -->
       </geometry>
-      <xacro:default_material/>
+      <xacro:default_material />
     </visual>
     <collision>
-      <origin rpy="0 0 3.1415926" xyz="0.047 0.0121 0.25"/>
+      <origin rpy="0 0 3.1415926" xyz="0.047 0.0121 0.25" />
       <geometry>
-        <mesh filename="package://smallrobot_description/meshes/link1.STL"/>
+        <mesh filename="package://smallrobot_description/meshes/link1.STL" />
       </geometry>
     </collision>
   </link>
   <joint name="joint1" type="revolute">
-    <origin rpy="0 0 0" xyz="0 0 0.043"/>
-    <axis xyz="0 0 1"/>
-    <limit effort="100" lower="-2.0" upper="2.0" velocity="1.57"/>
-    <parent link="base_link"/>
-    <child link="link1"/>
+    <origin rpy="0 0 0" xyz="0 0 0.043" />
+    <axis xyz="0 0 1" />
+    <limit effort="100" lower="-2.0" upper="2.0" velocity="1.57" />
+    <parent link="base_link" />
+    <child link="link1" />
   </joint>
   <link name="link1">
-    <xacro:default_inertial mass="0.5"/>
+    <xacro:default_inertial mass="0.5" />
     <visual>
-      <origin rpy="0 0 3.1415926" xyz="0.047 0.012 0.208"/>
+      <origin rpy="0 0 3.1415926" xyz="0.047 0.012 0.208" />
       <geometry>
-        <mesh filename="package://smallrobot_description/meshes/link2.STL"/>
+        <mesh filename="package://smallrobot_description/meshes/link2.STL" />
       </geometry>
-      <xacro:default_material/>
+      <xacro:default_material />
     </visual>
     <collision>
-      <origin rpy="0 0 3.1415926" xyz="0.047 0.012 0.208"/>
+      <origin rpy="0 0 3.1415926" xyz="0.047 0.012 0.208" />
       <geometry>
-        <mesh filename="package://smallrobot_description/meshes/link2.STL"/>
+        <mesh filename="package://smallrobot_description/meshes/link2.STL" />
       </geometry>
     </collision>
   </link>
   <joint name="joint2" type="revolute">
-    <origin rpy="0 0 0" xyz="0.047 -0.0485 0.098"/>
-    <axis xyz="0 1 0"/>
-    <limit effort="100" lower="-1.5707963" upper="3.1415926" velocity="1.57"/>
-    <parent link="link1"/>
-    <child link="link2"/>
+    <origin rpy="0 0 0" xyz="0.047 -0.0485 0.098" />
+    <axis xyz="0 1 0" />
+    <limit effort="100" lower="-1.5707963" upper="3.1415926" velocity="1.57" />
+    <parent link="link1" />
+    <child link="link2" />
   </joint>
   <link name="link2">
-    <xacro:default_inertial mass="0.3"/>
+    <xacro:default_inertial mass="0.3" />
     <visual>
-      <origin rpy="1.5707963 0 3.1415926" xyz="0 0 0"/>
+      <origin rpy="1.5707963 0 3.1415926" xyz="0 0 0" />
       <geometry>
-        <mesh filename="package://smallrobot_description/meshes/link3.STL"/>
+        <mesh filename="package://smallrobot_description/meshes/link3.STL" />
       </geometry>
-      <xacro:default_material/>
+      <xacro:default_material />
     </visual>
     <collision>
-      <origin rpy="1.5707963 0 3.1415926" xyz="0 0 0"/>
+      <origin rpy="1.5707963 0 3.1415926" xyz="0 0 0" />
       <geometry>
-        <mesh filename="package://smallrobot_description/meshes/link3.STL"/>
+        <mesh filename="package://smallrobot_description/meshes/link3.STL" />
       </geometry>
     </collision>
   </link>
   <joint name="joint3" type="revolute">
-    <origin rpy="0 0 0" xyz="0 0.08 0.111"/>
-    <axis xyz="0 1 0"/>
-    <limit effort="100" lower="-3.1415926" upper="1.5707963" velocity="1.57"/>
-    <parent link="link2"/>
-    <child link="link3"/>
+    <origin rpy="0 0 0" xyz="0 0.08 0.111" />
+    <axis xyz="0 1 0" />
+    <limit effort="100" lower="-3.1415926" upper="1.5707963" velocity="1.57" />
+    <parent link="link2" />
+    <child link="link3" />
   </joint>
   <link name="link3">
-    <xacro:default_inertial mass="0.1"/>
+    <xacro:default_inertial mass="0.1" />
     <visual>
-      <origin rpy="0 0 3.1415926" xyz="0.08 -0.0286 0.01"/>
+      <origin rpy="0 0 3.1415926" xyz="0.08 -0.0286 0.01" />
       <geometry>
-        <mesh filename="package://smallrobot_description/meshes/link4.STL"/>
+        <mesh filename="package://smallrobot_description/meshes/link4.STL" />
       </geometry>
-      <xacro:default_material/>
+      <xacro:default_material />
     </visual>
     <collision>
-      <origin rpy="0 0 3.1415926" xyz="0.08 -0.0286 0.01"/>
+      <origin rpy="0 0 3.1415926" xyz="0.08 -0.0286 0.01" />
       <geometry>
-        <mesh filename="package://smallrobot_description/meshes/link4.STL"/>
+        <mesh filename="package://smallrobot_description/meshes/link4.STL" />
       </geometry>
     </collision>
   </link>
   <joint name="joint4" type="revolute">
-    <origin rpy="0 1.5707963 0" xyz="-0.026 -0.0316 0.0258"/>
-    <axis xyz="0 0 1"/>
-    <limit effort="100" lower="-1.5707963" upper="1.5707963" velocity="1.57"/>
-    <parent link="link3"/>
-    <child link="link4"/>
+    <origin rpy="0 1.5707963 0" xyz="-0.026 -0.0316 0.0258" />
+    <axis xyz="0 0 1" />
+    <limit effort="100" lower="-1.5707963" upper="1.5707963" velocity="1.57" />
+    <parent link="link3" />
+    <child link="link4" />
   </joint>
   <link name="link4">
-    <xacro:default_inertial mass="0.1"/>
+    <xacro:default_inertial mass="0.1" />
     <visual>
-      <origin rpy="0 1.5707963 1.5707963" xyz="0.016 0.003 0.106"/>
+      <origin rpy="0 1.5707963 1.5707963" xyz="0.016 0.003 0.106" />
       <geometry>
         <mesh filename="package://smallrobot_description/meshes/link5.STL">
         </mesh>
       </geometry>
-      <xacro:default_material/>
+      <xacro:default_material />
     </visual>
     <collision>
-      <origin rpy="0 1.5707963 1.5707963" xyz="0.016 0.003 0.106"/>
+      <origin rpy="0 1.5707963 1.5707963" xyz="0.016 0.003 0.106" />
       <geometry>
-        <mesh filename="package://smallrobot_description/meshes/link5.STL"/>
+        <mesh filename="package://smallrobot_description/meshes/link5.STL" />
       </geometry>
     </collision>
   </link>
   <joint name="joint5" type="revolute">
-    <origin rpy="0 -1.5707963 0" xyz="0 0 0.144"/>
-    <axis xyz="0 1 0"/>
-    <limit effort="100" lower="-3.1415926" upper="3.1415926" velocity="1.57"/>
-    <parent link="link4"/>
-    <child link="link5"/>
+    <origin rpy="0 -1.5707963 0" xyz="0 0 0.144" />
+    <axis xyz="0 1 0" />
+    <limit effort="100" lower="-3.1415926" upper="3.1415926" velocity="1.57" />
+    <parent link="link4" />
+    <child link="link5" />
   </joint>
   <link name="link5">
-    <xacro:default_inertial mass="0.02"/>
+    <xacro:default_inertial mass="0.02" />
     <visual>
-      <origin rpy="3.1415926 0 -1.5707963" xyz="0.018 0 0"/>
+      <origin rpy="3.1415926 0 -1.5707963" xyz="0.018 0 0" />
       <geometry>
-        <mesh filename="package://smallrobot_description/meshes/link6.STL"/>
+        <mesh filename="package://smallrobot_description/meshes/link6.STL" />
       </geometry>
-      <xacro:default_material/>
+      <xacro:default_material />
     </visual>
     <collision>
-      <origin rpy="3.1415926 0 -1.5707963" xyz="0.018 0 0"/>
+      <origin rpy="3.1415926 0 -1.5707963" xyz="0.018 0 0" />
       <geometry>
-        <mesh filename="package://smallrobot_description/meshes/link6.STL"/>
+        <mesh filename="package://smallrobot_description/meshes/link6.STL" />
       </geometry>
     </collision>
   </link>
   <joint name="joint6" type="revolute">
-    <origin rpy="0 0 0" xyz="0.0253 0 0"/>
-    <axis xyz="1 0 0"/>
-    <limit effort="100" lower="-3.1415926" upper="3.1415926" velocity="1.57"/>
-    <parent link="link5"/>
-    <child link="link6"/>
+    <origin rpy="0 0 0" xyz="0.0253 0 0" />
+    <axis xyz="1 0 0" />
+    <limit effort="100" lower="-3.1415926" upper="3.1415926" velocity="1.57" />
+    <parent link="link5" />
+    <child link="link6" />
   </joint>
   <link name="link6">
-    <xacro:default_inertial mass="0.01"/>
+    <xacro:default_inertial mass="0.01" />
     <visual>
-      <origin rpy="0 0 3.1415926" xyz="-0.0555 0.003 -0.016"/>
+      <origin rpy="0 0 3.1415926" xyz="-0.0555 0.003 -0.016" />
       <geometry>
-        <mesh filename="package://smallrobot_description/meshes/link7.STL"/>
+        <mesh filename="package://smallrobot_description/meshes/link7.STL" />
       </geometry>
-      <xacro:default_material/>
+      <xacro:default_material />
     </visual>
     <collision>
-      <origin rpy="0 0 3.1415926" xyz="-0.0555 0.003 -0.016"/>
+      <origin rpy="0 0 3.1415926" xyz="-0.0555 0.003 -0.016" />
       <geometry>
-        <mesh filename="package://smallrobot_description/meshes/link7.STL"/>
+        <mesh filename="package://smallrobot_description/meshes/link7.STL" />
       </geometry>
     </collision>
   </link>
-  <xacro:default_transmission number='1' reduction_ratio='4.8'/>
-  <xacro:default_transmission number='2' reduction_ratio='4.0'/>
-  <xacro:default_transmission number='3' reduction_ratio='5.0'/>
-  <xacro:default_transmission number='4' reduction_ratio='2.8'/>
-  <xacro:default_transmission number='5' reduction_ratio='2.1'/>
-  <xacro:default_transmission number='6' reduction_ratio='1.0'/>
+  <link name="ee_link" />
+  <joint name="ee_fixed" type="fixed">
+    <parent link="link6" />
+    <child link="ee_link" />
+    <origin xyz="0 0 0.1" rpy="0 0 0" /> <!-- offset if needed -->
+  </joint>
+  <xacro:default_transmission number='1' reduction_ratio='4.8' />
+  <xacro:default_transmission number='2' reduction_ratio='4.0' />
+  <xacro:default_transmission number='3' reduction_ratio='5.0' />
+  <xacro:default_transmission number='4' reduction_ratio='2.8' />
+  <xacro:default_transmission number='5' reduction_ratio='2.1' />
+  <xacro:default_transmission number='6' reduction_ratio='1.0' />
 </robot>

File: src/smallrobot_description/urdf/smallrobot_ros2_control.xacro (robot description, xacro)
@@ -22,4 +22,5 @@
       </command_interface>
       <state_interface name="position" />
+      <state_interface name="velocity"/>
     </joint>
     <joint name="joint2">
@@ -29,4 +30,5 @@
       </command_interface>
       <state_interface name="position" />
+      <state_interface name="velocity"/>
     </joint>
     <joint name="joint3">
@@ -36,4 +38,5 @@
       </command_interface>
       <state_interface name="position" />
+      <state_interface name="velocity"/>
     </joint>
     <joint name="joint4">
@@ -43,4 +46,5 @@
       </command_interface>
       <state_interface name="position" />
+      <state_interface name="velocity"/>
     </joint>
     <joint name="joint5">
@@ -50,4 +54,5 @@
       </command_interface>
       <state_interface name="position" />
+      <state_interface name="velocity"/>
     </joint>
     <joint name="joint6">
@@ -57,4 +62,5 @@
       </command_interface>
       <state_interface name="position" />
+      <state_interface name="velocity"/>
     </joint>
   </ros2_control>

Commit message: add gripper for urdf

File: src/smallrobot_description/urdf/smallrobot.urdf.xacro (robot description, xacro)
@@ -7,15 +7,23 @@
 <robot xmlns:xacro="http://www.ros.org/wiki/xacro" name="smallrobot">
   <!-- PI & is_sim will be accessible from included xacro files -->
-  <xacro:arg name='is_sim' default='true' />
+  <xacro:arg name='is_sim'
+    default='true' />
   <xacro:property name='PI' value='3.14159' />
+  <xacro:property
+    name="meshes_file_direction"
+    value="package://smallrobot_description/meshes/" />
   <!-- include gazebo parameters -->
-  <xacro:include filename="$(find smallrobot_description)/urdf/smallrobot_gazebo.xacro" />
+  <xacro:include
+    filename="$(find smallrobot_description)/urdf/smallrobot_gazebo.xacro" />
   <!-- include ros2_control plugins -->
-  <xacro:include filename="$(find smallrobot_description)/urdf/smallrobot_ros2_control.xacro" />
+  <xacro:include
+    filename="$(find smallrobot_description)/urdf/smallrobot_ros2_control.xacro" />
   <!-- useful macros -->
-  <xacro:include filename="$(find smallrobot_description)/urdf/smallrobot_macro.xacro" />
+  <xacro:include
+    filename="$(find smallrobot_description)/urdf/smallrobot_macro.xacro" />
   <link name="world" />
   <!-- Fixed joint from world to base_link -->
-  <joint name="world_to_base" type="fixed">
+  <joint
+    name="world_to_base" type="fixed">
     <origin xyz="0 0 0" rpy="0 0 0" />
     <parent link="world" />
@@ -39,5 +47,6 @@
     </collision>
   </link>
-  <joint name="joint1" type="revolute">
+  <joint
+    name="joint1" type="revolute">
     <origin rpy="0 0 0" xyz="0 0 0.043" />
     <axis xyz="0 0 1" />
@@ -62,5 +71,6 @@
     </collision>
   </link>
-  <joint name="joint2" type="revolute">
+  <joint
+    name="joint2" type="revolute">
     <origin rpy="0 0 0" xyz="0.047 -0.0485 0.098" />
     <axis xyz="0 1 0" />
@@ -85,5 +95,6 @@
     </collision>
   </link>
-  <joint name="joint3" type="revolute">
+  <joint
+    name="joint3" type="revolute">
     <origin rpy="0 0 0" xyz="0 0.08 0.111" />
     <axis xyz="0 1 0" />
@@ -108,5 +119,6 @@
     </collision>
   </link>
-  <joint name="joint4" type="revolute">
+  <joint
+    name="joint4" type="revolute">
     <origin rpy="0 1.5707963 0" xyz="-0.026 -0.0316 0.0258" />
     <axis xyz="0 0 1" />
@@ -132,5 +144,6 @@
     </collision>
   </link>
-  <joint name="joint5" type="revolute">
+  <joint
+    name="joint5" type="revolute">
     <origin rpy="0 -1.5707963 0" xyz="0 0 0.144" />
     <axis xyz="0 1 0" />
@@ -163,5 +176,5 @@
   </joint>
   <link name="link6">
-    <xacro:default_inertial mass="0.01" />
+    <!-- <xacro:default_inertial mass="0.01" />
     <visual>
       <origin rpy="0 0 3.1415926" xyz="-0.0555 0.003 -0.016" />
@@ -176,12 +189,95 @@
         <mesh filename="package://smallrobot_description/meshes/link7.STL" />
       </geometry>
-    </collision>
-  </link>
-  <link name="ee_link" />
+    </collision> -->
+  </link>
+  <joint
+    name="gripper_left_joint" type="prismatic">
+    <parent link="link6" />
+    <child link="gripper_left_link" />
+    <origin xyz="0.0817 0.021 0.0" rpy="0 0 0" />
+    <axis xyz="0 1 0" />
+    <limit velocity="4.8" effort="1000" lower="-0.010" upper="0.019" />
+    <dynamics damping="0.1" />
+  </joint>
+  <link name="gripper_left_link">
+    <visual>
+      <origin xyz="-0.062 0 0" rpy="0 0 0" />
+      <geometry>
+        <mesh filename="${meshes_file_direction}/gripper_left_palm.stl" scale="0.001 0.001 0.001" />
+      </geometry>
+      <material name="grey">
+        <color rgba="0.2 0.2 0.2 1" />
+      </material>
+    </visual>
+    <collision>
+      <origin xyz="-0.062 0 0" rpy="0 0 0" />
+      <geometry>
+        <mesh filename="${meshes_file_direction}/gripper_left_palm.stl" scale="0.001 0.001 0.001" />
+      </geometry>
+    </collision>
+    <inertial>
+      <origin xyz="0 0 0" />
+      <mass value="1.0e-03" />
+      <inertia ixx="1.0e-06" ixy="0.0" ixz="0.0"
+        iyy="1.0e-06" iyz="0.0"
+        izz="1.0e-06" />
+    </inertial>
+  </link>
+  <joint name="gripper_right_joint" type="prismatic">
+    <parent link="link6" />
+    <child link="gripper_right_link" />
+    <origin xyz="0.0817 -0.021 0" rpy="0 0 0" />
+    <axis xyz="0 -1 0" />
+    <limit velocity="4.8" effort="1000" lower="-0.010" upper="0.019" />
+    <dynamics damping="0.7" />
+    <mimic joint="gripper_left_joint" multiplier="1" />
+  </joint>
+  <link
+    name="gripper_right_link">
+    <visual>
+      <origin xyz="-0.062 0 0" rpy="0 0 0" />
+      <geometry>
+        <mesh filename="${meshes_file_direction}/gripper_right_palm.stl" scale="0.001 0.001 0.001" />
+      </geometry>
+      <material name="grey">
+        <color rgba="0.2 0.2 0.2 1" />
+      </material>
+    </visual>
+    <collision>
+      <origin xyz="-0.062 0 0" rpy="0 0 0" />
+      <geometry>
+        <mesh filename="${meshes_file_direction}/gripper_right_palm.stl" scale="0.001 0.001 0.001" />
+      </geometry>
+    </collision>
+    <inertial>
+      <origin xyz="0 0 0" />
+      <mass value="1.0e-03" />
+      <inertia ixx="1.0e-06" ixy="0.0" ixz="0.0"
+        iyy="1.0e-06" iyz="0.0"
+        izz="1.0e-06" />
+    </inertial>
+  </link>
+  <joint name="end_effector_joint" type="fixed">
+    <parent link="link6" />
+    <child link="end_effector_link" />
+    <origin xyz="0.126 0.0 0.0" rpy="0 0 0" />
+  </joint>
+  <link name="end_effector_link">
+    <visual>
+      <origin xyz="-0.05 0 0" rpy="0 0 0" />
+      <geometry>
+        <box size="0.01 0.01 0.01" />
+      </geometry>
+      <material name="red">
+        <color rgba="1.0 0.0 0.0 1" />
+      </material>
+    </visual>
+  </link>
+  <!-- <link name="ee_link" />
   <joint name="ee_fixed" type="fixed">
     <parent link="link6" />
     <child link="ee_link" />
-    <origin xyz="0 0 0.1" rpy="0 0 0" /> <!-- offset if needed -->
-  </joint>
+    <origin xyz="0 0 0.1" rpy="0 0 0" />
+  </joint> -->
   <xacro:default_transmission number='1' reduction_ratio='4.8' />
   <xacro:default_transmission number='2' reduction_ratio='4.0' />
