Commit message: FIX: moveit2 works for gripper

File: src/smallrobot_description/urdf/smallrobot.urdf.xacro (robot description, xacro)
@@ -287,27 +287,17 @@
     </inertial>
   </link>
-  <!--
   <joint name="end_effector_joint" type="fixed">
-    <parent link="link6" />
+    <parent link="flange" />
     <child link="end_effector_link" />
-    <origin xyz="0.126 0.0 0.0" rpy="0 0 0" />
+    <origin xyz="0.05 0.0 0.0" rpy="0 0 0" />
   </joint>
   <link name="end_effector_link">
-    <visual>
-      <origin xyz="-0.05 0 0" rpy="0 0 0" />
-      <geometry>
-        <box size="0.01 0.01 0.01" />
-      </geometry>
-      <material name="red">
-        <color rgba="1.0 0.0 0.0 1" />
-      </material>
-    </visual>
-  </link> -->
+  </link>
   <!-- <link name="ee_link" />
   <joint name="ee_fixed" type="fixed">
-    <parent link="link6" />
+    <parent link="flange" />
     <child link="ee_link" />
     <origin xyz="0 0 0.1" rpy="0 0 0" />
-  </joint> -->
+  </joint>  -->
   <xacro:default_transmission idx='1' joint_name='joint1' reduction_ratio='4.8' />
   <xacro:default_transmission idx='2' joint_name='joint2' reduction_ratio='4.0' />

File: src/smallrobot_description/urdf/smallrobot_ros2_control.xacro (robot description, xacro)
@@ -70,5 +70,5 @@
       </command_interface>
       <state_interface name="position" />
-      <!-- <state_interface name="velocity"/> -->
+      <state_interface name="velocity"/>
     </joint>
     <joint name="gripper_right_joint">
@@ -80,5 +80,5 @@
       </command_interface>
       <state_interface name="position" />
-      <!-- <state_interface name="velocity"/> -->
+      <state_interface name="velocity"/>
     </joint>
   </ros2_control>

File: src/smallrobot_moveit/config/smallrobot.ros2_control.xacro (robot description, xacro)
@@ -50,4 +50,11 @@
                 <state_interface name="velocity"/>
             </joint>
+            <joint name="gripper_left_joint">
+                <command_interface name="position"/>
+                <state_interface name="position">
+                  <param name="initial_value">${initial_positions['gripper_left_joint']}</param>
+                </state_interface>
+                <state_interface name="velocity"/>
+            </joint>
         </ros2_control>
     </xacro:macro>

File: src/smallrobot_moveit/config/smallrobot.urdf.xacro (robot description, xacro)
@@ -3,5 +3,5 @@
     <xacro:arg name="initial_positions_file" default="initial_positions.yaml" />
     <!-- Import smallrobot urdf file -->
-    <xacro:include filename="$(find smallrobot_description)/urdf/smallrobot.urdf" />
+    <xacro:include filename="$(find smallrobot_description)/urdf/smallrobot.urdf.xacro" />
     <!-- Import control_xacro -->
     <xacro:include filename="smallrobot.ros2_control.xacro" />

Commit message: FIX: gazebo sim ok. refence to open_manipulator, use mocK_compoents/GenericSystem plugin , add empty_world.world, refer to turtlebot3_gazebo/worlds/empty_world.world

File: src/smallrobot_description/urdf/smallrobot.urdf.xacro (robot description, xacro)
@@ -300,11 +300,3 @@
     <origin xyz="0 0 0.1" rpy="0 0 0" />
   </joint>  -->
-  <xacro:default_transmission idx='1' joint_name='joint1' reduction_ratio='4.8' />
-  <xacro:default_transmission idx='2' joint_name='joint2' reduction_ratio='4.0' />
-  <xacro:default_transmission idx='3' joint_name='joint3' reduction_ratio='5.0' />
-  <xacro:default_transmission idx='4' joint_name='joint4' reduction_ratio='2.8' />
-  <xacro:default_transmission idx='5' joint_name='joint5' reduction_ratio='2.1' />
-  <xacro:default_transmission idx='6' joint_name='joint6' reduction_ratio='1.0' />
-  <xacro:default_transmission idx='7' joint_name='gripper_left_joint' reduction_ratio='1.0' />
-  <xacro:default_transmission idx='8' joint_name='gripper_right_joint' reduction_ratio='1.0' />
 </robot>

File: src/smallrobot_description/urdf/smallrobot_gazebo.xacro (robot description, xacro)
@@ -1,10 +1,22 @@
 <?xml version="1.0"?>
 <robot xmlns:xacro="http://www.ros.org/wiki/xacro" name="smallrobot" params="number">
+    <xacro:macro name="default_transmission" params="idx joint_name reduction_ratio">
+        <transmission name="transmission_${idx}">
+        <type>transmission_interface/SimpleTransmission</type>
+        <actuator name="motor_${idx}">
+            <mechanicalReduction>${reduction_ratio}</mechanicalReduction>
+        </actuator>
+        <joint name="${joint_name}">
+            <hardwareInterface>hardware_interface/position</hardwareInterface>
+            <hardwareInterface>hardware_interface/velocity</hardwareInterface>
+            <!-- <hardwareInterface>hardware_interface/effort</hardwareInterface> -->
+        </joint>
+        </transmission>
+    </xacro:macro>
     <gazebo>
-        <plugin name="gazebo_ros2_control" filename="libgazebo_ros2_control.so">
-            <robot_param>robot_description</robot_param>
-            <robot_param_node>robot_state_publisher</robot_param_node>
-            <!-- <parameters>/home/roach/ros2_ws/install/robotarm_controller/share/robotarm_controller/config/robotarm_controllers.yaml</parameters> -->
-            <parameters>$(find robotarm_controller)/config/robotarm_controllers.yaml</parameters>
+        <plugin filename="gz_ros2_control-system" name="gz_ros2_control::GazeboSimROS2ControlPlugin">
+            <!-- <robot_param>robot_description</robot_param>
+            <robot_param_node>robot_state_publisher</robot_param_node>   -->
+            <parameters>$(find robotarm_controller)/config/sim_controllers.yaml</parameters>
         </plugin>
     </gazebo>
@@ -36,3 +48,14 @@
         <material>Gazebo/Grey</material>
     </gazebo>
+    <gazebo reference='end_effector_link'>
+        <material>Gazebo/Black</material>
+    </gazebo>
+    <xacro:default_transmission idx='1' joint_name='joint1' reduction_ratio='4.8' />
+    <xacro:default_transmission idx='2' joint_name='joint2' reduction_ratio='4.0' />
+    <xacro:default_transmission idx='3' joint_name='joint3' reduction_ratio='5.0' />
+    <xacro:default_transmission idx='4' joint_name='joint4' reduction_ratio='2.8' />
+    <xacro:default_transmission idx='5' joint_name='joint5' reduction_ratio='2.1' />
+    <xacro:default_transmission idx='6' joint_name='joint6' reduction_ratio='1.0' />
+    <xacro:default_transmission idx='7' joint_name='gripper_left_joint' reduction_ratio='1.0' />
+    <xacro:default_transmission idx='8' joint_name='gripper_right_joint' reduction_ratio='1.0' />
 </robot>

File: src/smallrobot_description/urdf/smallrobot_macro.xacro (robot description, xacro)
@@ -10,17 +10,4 @@
         izz="${m*r*r/2}" /> -->
     </inertial>
-  </xacro:macro>
-  <xacro:macro name="default_transmission" params="idx joint_name reduction_ratio">
-    <transmission name="transmission_${idx}">
-      <type>transmission_interface/SimpleTransmission</type>
-      <actuator name="motor_${idx}">
-        <mechanicalReduction>${reduction_ratio}</mechanicalReduction>
-      </actuator>
-      <joint name="${joint_name}">
-        <hardwareInterface>hardware_interface/position</hardwareInterface>
-        <hardwareInterface>hardware_interface/velocity</hardwareInterface>
-        <!-- <hardwareInterface>hardware_interface/effort</hardwareInterface> --> -->
-      </joint>
-    </transmission>
   </xacro:macro>
   <xacro:macro name="default_material">

File: src/smallrobot_description/urdf/smallrobot_ros2_control.xacro (robot description, xacro)
@@ -5,7 +5,8 @@
     <!-- ros2_control gazebo simulator-->
     <xacro:if value="$(arg is_sim)">
-      <hardware>
-        <plugin>gazebo_ros2_control/GazeboSystem</plugin>
-      </hardware>
+       <hardware>
+          <!-- <plugin>gz_ros2_control/GazeboSimSystem</plugin> -->
+          <plugin>mock_components/GenericSystem</plugin>
+        </hardware>
     </xacro:if>
     <!-- ros2_control real robot hw interface-->
@@ -72,14 +73,6 @@
       <state_interface name="velocity"/>
     </joint>
-    <joint name="gripper_right_joint">
-      <!-- <param name='mimic'>gripper_left_joint</param>
-      <param name='multiplier'>1.0</param> -->
-      <command_interface name="position">
-        <param name='min'>-0.01</param>
-        <param name='max'>0.019</param>
-      </command_interface>
-      <state_interface name="position" />
-      <state_interface name="velocity"/>
-    </joint>
+    <!-- <joint name="gripper_right_joint">
+    </joint> -->
   </ros2_control>
 </robot>

Commit message: bugfix by amazonQ - sim is ok. add inertial and mass

File: src/smallrobot_description/urdf/smallrobot.urdf.xacro (robot description, xacro)
@@ -32,5 +32,5 @@
   </joint>
   <link name="base_link">
-    <xacro:default_inertial mass="1.0" />
+    <xacro:base_inertial mass="2.5" />
     <visual>
       <origin rpy="0 0 ${PI}" xyz="0.047 0.0121 0.25" />
@@ -57,5 +57,5 @@
   </joint>
   <link name="link1">
-    <xacro:default_inertial mass="0.5" />
+    <xacro:link1_inertial mass="1.2" />
     <visual>
       <origin rpy="0 0 ${PI}" xyz="0.047 0.012 0.208" />
@@ -81,5 +81,5 @@
   </joint>
   <link name="link2">
-    <xacro:default_inertial mass="0.3" />
+    <xacro:link2_inertial mass="0.8" />
     <visual>
       <origin rpy="${PI/2} 0 ${PI}" xyz="0 0 0" />
@@ -105,5 +105,5 @@
   </joint>
   <link name="link3">
-    <xacro:default_inertial mass="0.1" />
+    <xacro:link3_inertial mass="0.3" />
     <visual>
       <origin rpy="0 0 ${PI}" xyz="0.08 -0.0286 0.01" />
@@ -129,5 +129,5 @@
   </joint>
   <link name="link4">
-    <xacro:default_inertial mass="0.1" />
+    <xacro:link4_inertial mass="0.25" />
     <visual>
       <origin rpy="0 ${PI/2} ${PI/2}" xyz="0.016 0.003 0.106" />
@@ -153,5 +153,5 @@
   </joint>
   <link name="link5">
-    <xacro:default_inertial mass="0.02" />
+    <xacro:link5_inertial mass="0.15" />
     <visual>
       <origin rpy="${PI} 0 -${PI/2}" xyz="0.018 0 0" />
@@ -176,5 +176,5 @@
   </joint>
   <link name="link6">
-    <xacro:default_inertial mass="0.01" />
+    <xacro:link6_inertial mass="0.1" />
     <visual>
       <origin rpy="0 0 ${PI}" xyz="-0.0555 0.003 -0.016" />
@@ -260,5 +260,4 @@
     <limit acceleration="2.0" velocity="04.8" effort="10" lower="-0.010" upper="0.019" />
     <dynamics damping="0.7" />
-    <mimic joint="gripper_left_joint" multiplier="1" />
   </joint>
   <link
@@ -300,3 +299,5 @@
     <origin xyz="0 0 0.1" rpy="0 0 0" />
   </joint>  -->
+  <!-- Activate Gazebo plugin -->
+  <xacro:smallrobot_gazebo />
 </robot>

File: src/smallrobot_description/urdf/smallrobot_gazebo.xacro (robot description, xacro)
@@ -60,9 +60,7 @@
     <gazebo>
         <plugin filename="gz_ros2_control-system" name="gz_ros2_control::GazeboSimROS2ControlPlugin">
+            <robot_param>robot_description</robot_param>
+            <robot_param_node>robot_state_publisher</robot_param_node>
             <parameters>$(find robotarm_controller)/config/sim_controllers.yaml</parameters>
-            <ros>
-                <remapping>/controller_manager/robot_description:=/robot_description</remapping>
-            </ros>
-            <!-- <controller_manager_prefix_node_name>controller_manager</controller_manager_prefix_node_name> -->
         </plugin>
     </gazebo>

File: src/smallrobot_description/urdf/smallrobot_macro.xacro (robot description, xacro)
@@ -6,7 +6,68 @@
       <mass value="${mass}" />
       <inertia ixx="1.0" ixy="0" ixz="0" iyy="1.0" iyz="0" izz="1.0" />
-      <!-- for cylinder robort formular in wiki <inertia ixx="${m*(3*r*r+h*h)/12}" ixy="0" ixz="0"
-      iyy="${m*(3*r*r+h*h)/12}" iyz="0"
-        izz="${m*r*r/2}" /> -->
+    </inertial>
+  </xacro:macro>
+  <!-- Accurate inertial properties for robot links -->
+  <xacro:macro name="base_inertial" params="mass">
+    <inertial>
+      <origin xyz="0.047 0.0121 0.125" rpy="0 0 0"/>
+      <mass value="${mass}" />
+      <inertia ixx="${mass*0.083}" ixy="0.001" ixz="0.002"
+               iyy="${mass*0.083}" iyz="0.001"
+               izz="${mass*0.025}" />
+    </inertial>
+  </xacro:macro>
+  <xacro:macro name="link1_inertial" params="mass">
+    <inertial>
+      <origin xyz="0.047 0.012 0.104" rpy="0 0 0"/>
+      <mass value="${mass}" />
+      <inertia ixx="${mass*0.045}" ixy="0.001" ixz="0.001"
+               iyy="${mass*0.045}" iyz="0.001"
+               izz="${mass*0.015}" />
+    </inertial>
+  </xacro:macro>
+  <xacro:macro name="link2_inertial" params="mass">
+    <inertial>
+      <origin xyz="0 0.04 0.055" rpy="0 0 0"/>
+      <mass value="${mass}" />
+      <inertia ixx="${mass*0.012}" ixy="0" ixz="0"
+               iyy="${mass*0.025}" iyz="0.002"
+               izz="${mass*0.020}" />
+    </inertial>
+  </xacro:macro>
+  <xacro:macro name="link3_inertial" params="mass">
+    <inertial>
+      <origin xyz="-0.013 -0.015 0.013" rpy="0 0 0"/>
+      <mass value="${mass}" />
+      <inertia ixx="${mass*0.003}" ixy="0" ixz="0"
+               iyy="${mass*0.008}" iyz="0"
+               izz="${mass*0.008}" />
+    </inertial>
+  </xacro:macro>
+  <xacro:macro name="link4_inertial" params="mass">
+    <inertial>
+      <origin xyz="0.008 0.001 0.072" rpy="0 0 0"/>
+      <mass value="${mass}" />
+      <inertia ixx="${mass*0.018}" ixy="0" ixz="0"
+               iyy="${mass*0.018}" iyz="0"
+               izz="${mass*0.002}" />
+    </inertial>
+  </xacro:macro>
+  <xacro:macro name="link5_inertial" params="mass">
+    <inertial>
+      <origin xyz="0.009 0 0" rpy="0 0 0"/>
+      <mass value="${mass}" />
+      <inertia ixx="${mass*0.001}" ixy="0" ixz="0"
+               iyy="${mass*0.002}" iyz="0"
+               izz="${mass*0.002}" />
+    </inertial>
+  </xacro:macro>
+  <xacro:macro name="link6_inertial" params="mass">
+    <inertial>
+      <origin xyz="-0.028 0.002 -0.008" rpy="0 0 0"/>
+      <mass value="${mass}" />
+      <inertia ixx="${mass*0.001}" ixy="0" ixz="0"
+               iyy="${mass*0.003}" iyz="0"
+               izz="${mass*0.003}" />
     </inertial>
   </xacro:macro>

Commit message: FIX: Removing controller manager node since Gazebo plugin handles it in simulation.

File: src/smallrobot_description/urdf/smallrobot.urdf.xacro (robot description, xacro)
@@ -36,5 +36,5 @@
       <origin rpy="0 0 ${PI}" xyz="0.047 0.0121 0.25" />
       <geometry>
-        <mesh filename="package://smallrobot_description/meshes/link1.STL" />
+        <mesh filename="${meshes_file_direction}/link1.STL" />
         <!-- <box size="0.5 0.5 0.5"/> -->
       </geometry>
@@ -44,5 +44,5 @@
       <origin rpy="0 0 ${PI}" xyz="0.047 0.0121 0.25" />
       <geometry>
-        <mesh filename="package://smallrobot_description/meshes/link1.STL" />
+        <mesh filename="${meshes_file_direction}/link1.STL" />
       </geometry>
     </collision>
@@ -61,5 +61,5 @@
       <origin rpy="0 0 ${PI}" xyz="0.047 0.012 0.208" />
       <geometry>
-        <mesh filename="package://smallrobot_description/meshes/link2.STL" />
+        <mesh filename="${meshes_file_direction}/link2.STL" />
       </geometry>
       <xacro:default_material />
@@ -68,5 +68,5 @@
       <origin rpy="0 0 ${PI}" xyz="0.047 0.012 0.208" />
       <geometry>
-        <mesh filename="package://smallrobot_description/meshes/link2.STL" />
+        <mesh filename="${meshes_file_direction}/link2.STL" />
       </geometry>
     </collision>
@@ -85,5 +85,5 @@
       <origin rpy="${PI/2} 0 ${PI}" xyz="0 0 0" />
       <geometry>
-        <mesh filename="package://smallrobot_description/meshes/link3.STL" />
+        <mesh filename="${meshes_file_direction}/link3.STL" />
       </geometry>
       <xacro:default_material />
@@ -92,5 +92,5 @@
       <origin rpy="${PI/2} 0 ${PI}" xyz="0 0 0" />
       <geometry>
-        <mesh filename="package://smallrobot_description/meshes/link3.STL" />
+        <mesh filename="${meshes_file_direction}/link3.STL" />
       </geometry>
     </collision>
@@ -109,5 +109,5 @@
       <origin rpy="0 0 ${PI}" xyz="0.08 -0.0286 0.01" />
       <geometry>
-        <mesh filename="package://smallrobot_description/meshes/link4.STL" />
+        <mesh filename="${meshes_file_direction}/link4.STL" />
       </geometry>
       <xacro:default_material />
@@ -116,5 +116,5 @@
       <origin rpy="0 0 ${PI}" xyz="0.08 -0.0286 0.01" />
       <geometry>
-        <mesh filename="package://smallrobot_description/meshes/link4.STL" />
+        <mesh filename="${meshes_file_direction}/link4.STL" />
       </geometry>
     </collision>
@@ -133,6 +133,5 @@
       <origin rpy="0 ${PI/2} ${PI/2}" xyz="0.016 0.003 0.106" />
       <geometry>
-        <mesh filename="package://smallrobot_description/meshes/link5.STL">
-        </mesh>
+        <mesh filename="${meshes_file_direction}/link5.STL" />
       </geometry>
       <xacro:default_material />
@@ -141,5 +140,5 @@
       <origin rpy="0 ${PI/2} ${PI/2}" xyz="0.016 0.003 0.106" />
       <geometry>
-        <mesh filename="package://smallrobot_description/meshes/link5.STL" />
+        <mesh filename="${meshes_file_direction}/link5.STL" />
       </geometry>
     </collision>
@@ -157,5 +156,5 @@
       <origin rpy="${PI} 0 -${PI/2}" xyz="0.018 0 0" />
       <geometry>
-        <mesh filename="package://smallrobot_description/meshes/link6.STL" />
+        <mesh filename="${meshes_file_direction}/link6.STL" />
       </geometry>
       <xacro:default_material />
@@ -164,5 +163,5 @@
       <origin rpy="${PI} 0 -${PI/2}" xyz="0.018 0 0" />
       <geometry>
-        <mesh filename="package://smallrobot_description/meshes/link6.STL" />
+        <mesh filename="${meshes_file_direction}/link6.STL" />
       </geometry>
     </collision>
@@ -180,5 +179,5 @@
       <origin rpy="0 0 ${PI}" xyz="-0.0555 0.003 -0.016" />
       <geometry>
-        <mesh filename="package://smallrobot_description/meshes/link7.STL" />
+        <mesh filename="${meshes_file_direction}/link7.STL" />
       </geometry>
       <xacro:default_material />
@@ -187,5 +186,5 @@
       <origin rpy="0 0 ${PI}" xyz="-0.0555 0.003 -0.016" />
       <geometry>
-        <mesh filename="package://smallrobot_description/meshes/link7.STL" />
+        <mesh filename="${meshes_file_direction}/link7.STL" />
       </geometry>
     </collision>
@@ -260,4 +259,7 @@
     <limit acceleration="2.0" velocity="04.8" effort="10" lower="-0.010" upper="0.019" />
     <dynamics damping="0.7" />
+    <xacro:unless value="$(arg is_sim)">
+      <mimic joint="gripper_left_joint" multiplier="1" />
+    </xacro:unless>
   </joint>
   <link

File: src/smallrobot_description/urdf/smallrobot_gazebo.xacro (robot description, xacro)
@@ -17,22 +17,43 @@
     <gazebo reference="base_link">
         <material>Gazebo/White</material>
+        <mu1>0.2</mu1>
+        <mu2>0.2</mu2>
+        <self_collide>0</self_collide>
     </gazebo>
     <gazebo reference="link1">
         <material>Gazebo/Orange</material>
+        <mu1>0.2</mu1>
+        <mu2>0.2</mu2>
+        <self_collide>0</self_collide>
     </gazebo>
      <gazebo reference="link2">
         <material>Gazebo/Orange</material>
+        <mu1>0.2</mu1>
+        <mu2>0.2</mu2>
+        <self_collide>0</self_collide>
     </gazebo>
      <gazebo reference="link3">
         <material>Gazebo/Orange</material>
+        <mu1>0.2</mu1>
+        <mu2>0.2</mu2>
+        <self_collide>0</self_collide>
     </gazebo>
      <gazebo reference="link4">
         <material>Gazebo/Orange</material>
+        <mu1>0.2</mu1>
+        <mu2>0.2</mu2>
+        <self_collide>0</self_collide>
     </gazebo>
     <gazebo reference="link5">
-        <material>Gazebo/Orange</material>
+        <material>Gazebo/White</material>
+        <mu1>0.2</mu1>
+        <mu2>0.2</mu2>
+        <self_collide>0</self_collide>
     </gazebo>
     <gazebo reference="link6">
         <material>Gazebo/Orange</material>
+        <mu1>0.2</mu1>
+        <mu2>0.2</mu2>
+        <self_collide>0</self_collide>
     </gazebo>
     <gazebo reference="gripper_left_link">
@@ -60,6 +81,4 @@
     <gazebo>
         <plugin filename="gz_ros2_control-system" name="gz_ros2_control::GazeboSimROS2ControlPlugin">
-            <robot_param>robot_description</robot_param>
-            <robot_param_node>robot_state_publisher</robot_param_node>
             <parameters>$(find robotarm_controller)/config/sim_controllers.yaml</parameters>
         </plugin>

File: src/smallrobot_description/urdf/smallrobot_ros2_control.xacro (robot description, xacro)
@@ -72,6 +72,8 @@
       <state_interface name="velocity"/>
     </joint>
-    <!-- <joint name="gripper_right_joint">
-    </joint> -->
+    <joint name="gripper_right_joint">
+      <state_interface name="position" />
+      <state_interface name="velocity"/>
+    </joint>
   </ros2_control>
 </robot>
