Commit message: amend: update_rate: 50hz from 10hz

File: src/smallrobot_description/urdf/smallrobot_updated.urdf (robot description, URDF)
Before this commit: robot smallrobot, 12 links, 11 joints
Joints:
- joint joint2: limit lower=-1.570795 upper=3.14159 effort=10 velocity=4.8 -> lower=-1.5707963 upper=3.1415926 effort=100 velocity=0.4
- joint joint6: limit lower=-3.14159 upper=3.14159 effort=10 velocity=4.8 -> lower=-3.1415926 upper=3.1415926 effort=100 velocity=0.4
